File: mini-pcb/stm32f0-can-mini-breakout.kicad_pcb (KiCad board)
At the start: 2 copper layers, 103.8 x 53.7 mm, 116 parts, among them J1 POWER_BUS, J10 I2C, J11 GS2, J12 Conn_01x02, J13 Conn_01x09, J14 Conn_01x09, J15 Conn_01x09, J16 Conn_01x09, J17 Conn_01x09, J18 Conn_01x09, J19 Conn_01x08, J2 POWER_BUS, J20 Conn_01x08, J21 Conn_01x08, J22 Conn_01x05, J23 Conn_01x05, J24 Conn_01x05, J25 Conn_01x05, J26 Conn_01x09, J27 Conn_01x09, J28 Conn_01x09, J29 Conn_01x07, J3 GS2, J30 Conn_01x09, J31 Conn_01x09, J32 Conn_01x09, J33 Conn_01x09, J34 Conn_01x07, J35 Conn_01x10, J36 USB, J37 Conn_01x09, J38 Conn_01x09, J39 Conn_01x05, J4 GS2, J40 Conn_01x05, J41 Conn_01x07, J43 Conn_01x05, J44 Conn_01x05, J45 Conn_01x05, J46 Screw_Terminal_01x02, J47 Screw_Terminal_01x02, J48 Screw_Terminal_01x02, J49 Screw_Terminal_01x02, J5 GS2, J6 UART, J7 SWD, J8 STEPDOWN, J9 I2C, Q1 N-FET, Q10 BT138-800, Q11 BT138-800, Q12 BT138-800, Q2 N-FET, Q3 N-FET, Q4 N-FET, Q5 N-FET, Q6 N-FET, Q7 N-FET, Q8 N-FET, Q9 BT138-800, U1 AT24CS64-SSHM, U2 SN65HVD230, U3 STM32F072C8Tx, U4 MOC3063M, U5 MOC3063M, U6 MOC3063M, U7 MOC3063M, Y1 Crystal

Commit message: update pcb
Other:
- rule pad_to_mask_clearance: 0.2 -> 0.05
Changed lines of the file:
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@@
     (links 231)
     (no_connects 0)
-    (area 60.924999 21.824999 164.875001 75.675001)
+    (area 56.7028 18.521427 170.857143 77.319)
     (thickness 1.6)
     (drawings 56)
@@
     (pad_size 1.524 1.524)
     (pad_drill 0.762)
-    (pad_to_mask_clearance 0.2)
+    (pad_to_mask_clearance 0.05)
+    (solder_mask_min_width 0.15)
     (aux_axis_origin 0 0)
     (visible_elements FFFFFF7F)
     (pcbplotparams
-      (layerselection 0x00030_80000001)
+      (layerselection 0x010f0_80000001)
       (usegerberextensions false)
       (excludeedgelayer true)
