File: pcb/base_heating.sch (KiCad schematic (older format))
At the start: 80 parts, among them J1 X1_1-20, J10 I2C, J11 USB, J12 POWER_BUS, J13 POWER_BUS, J14 DCSW_2, J15 DCSW_1, J16 ACSW_1, J17 RS422, J2 X1_21-40, J3 STEPDOWN, J4 BOOT, J5 GND, J6 DIN_1, J7 SWD, J8 I2C, J9 A_D_IN, Q1 NTR2101P, Q2 IRF540N, Q3 IRF540N, Q4 IRF540N, Q5 IRF540N, Q6 BT136, U1 MAX3078E, U2 SN65HVD230, U3 AT24CS64-SSHM, U4 STM32F072C8Tx, U5 MOC3061M, U6 MOC3061M

Commit message: Finished schematics, updated screenshot
Parts:
- added J18: UART_1, Pin_Headers:Pin_Header_Straight_1x03, symbol Conn_01x03
- added JP1, JP2, JP3: Jumper_NO_Small, Capacitors_SMD:C_0201_NoSilk, symbol Jumper_NO_Small
- added Q7: BT136, TO_SOT_Packages_THT:TO-220_Neutral123_Vertical, symbol BT136-800
- added R28: 360, Resistors_SMD:R_0805_HandSoldering, symbol R
- added R29, R30: 38, Resistors_THT:R_Axial_DIN0207_L6.3mm_D2.5mm_P5.08mm_Vertical, symbol R
- C16: value 100n -> 10n; footprint Capacitors_SMD:C_0805_HandSoldering -> Capacitors_THT:C_Rect_L7.0mm_W6.5mm_P5.00mm
- C17: footprint Capacitors_ThroughHole:C_Rect_L7.5_W6.5_P5 -> Capacitors_THT:C_Rect_L7.0mm_W6.5mm_P5.00mm
- R19: value 0 -> 10k
- R20: value 10k -> 360
- R26, R27: footprint Resistors_ThroughHole:Resistor_Vertical_RM5mm -> Resistors_THT:R_Axial_DIN0207_L6.3mm_D2.5mm_P5.08mm_Vertical
Connections:
- net DIN5 is gone; now on net AIN_FB1: J9.1 (Pin_1)
- net DIN_SENSE is gone; now on net ACSW_1: J1.12 (Pin_12)
- net DIN_SW_B3_246 is gone; now on net DIN1: J2.11 (Pin_11)
- net DOUT_LED_GREEN is gone; now on net ACSW_2: J2.7 (Pin_7)
- net DOUT_SW_C12 is gone; now on net DIN4: J2.8 (Pin_8)
- net DOUT_SW_C34 is gone; now on net DIN3: J2.9 (Pin_9)
- net DOUT_SW_C56 is gone; now on net DIN2: J2.10 (Pin_10)
- net LED_A is gone; now on net DOUT_LED_RED: R4.1
- net LED_B is gone; now on net DOUT_K6_20B: R5.1
- net ODSW_3 is gone; now on net DIN_SW_B1_135: Q3.1 (G)
- net ODSW_4 is gone; now on net DIN_SW_B3_135: Q2.1 (G)
- net RS422DE is gone; now on net AIN_ATS: U1.3 (DE)
- net RS422RE is gone; now on net GND: U1.2 (~RE~)
- net USB_DM is gone; now on net DOUT_K2_20A: J11.2 (Pin_2), U4.32 (CAN_RX/COMP1_OUT/TIM1_CH4/TSC_G4_IO3/USART1_CTS/USB_DM/PA11)
- net USB_DP is gone; now on net DOUT_K1_FIRE: J11.1 (Pin_1), U4.33 (CAN_TX/COMP2_OUT/TIM1_ETR/TSC_G4_IO4/USART1_DE/USART1_RTS/USB_DP/PA12)
- net +3V3: now also J17.4 (Pin_4), JP1.1, JP2.1, JP3.1
- net ACSW_1: now also U4.22 (PB11/I2C2_SDA/TIM2_CH4/TSC_G6_IO1/USART3_RX)
- net ACSW_2: now also U4.18 (PB0/ADC_IN8/TIM1_CH2N/TIM3_CH3/TSC_G3_IO2/USART3_CK)
- net AIN_ATS: now also R19.2
- net AIN_A_D: now also C3.1, J1.2 (Pin_2), J9.4 (Pin_4), R1.2, R7.2; no longer R19.2, U4.17 (ADC_IN7/COMP2_OUT/I2S1_SD/SPI1_MOSI/TIM14_CH1/TIM17_CH1/TIM1_CH1N/TIM3_CH2/TSC_G2_IO4/PA7)
- net AIN_KTS: now also U1.4 (DI)
- net AIN_VTS: now also U1.1 (RO)
- net CAN_SUSPEND: now also U4.2 (PC13/RTC_OUT_ALARM/RTC_OUT_CALIB/RTC_TAMP1/RTC_TS/SYS_WKUP2)
- net DIN1: now also U4.6 (PF1/RCC_OSC_OUT)
- net DIN2: now also U4.21 (PB10/CEC/I2C2_SCL/I2S2_CK/SPI2_SCK/TIM2_CH3/TSC_SYNC/USART3_TX)
- net DIN3: now also U4.20 (PB2/TSC_G3_IO4)
- net DIN4: now also U4.19 (PB1/ADC_IN9/TIM14_CH1/TIM1_CH3N/TIM3_CH4/TSC_G3_IO3/USART3_DE/USART3_RTS)
- net DIN_SW_B0_135: now also U4.27 (PB14/I2C2_SDA/I2S2_MCK/SPI2_MISO/TIM15_CH1/TIM1_CH2N/TSC_G6_IO4/USART3_DE/USART3_RTS)
- net DIN_SW_B0_246: now also U4.3 (PC14/RCC_OSC32_IN)
- net DIN_SW_B1_135: now also U4.29 (CRS_SYNC/RCC_MCO/TIM1_CH1/USART1_CK/PA8)
- net DIN_SW_B1_246: now also U4.4 (PC15/RCC_OSC32_OUT)
- net DIN_SW_B2_135: now also U4.31 (TIM17_BKIN/TIM1_CH3/TSC_G4_IO2/USART1_RX/PA10), J18.2 (Pin_2)
- net DIN_SW_B2_246: now also U4.5 (PF0/CRS_SYNC/RCC_OSC_IN)
- net DIN_SW_B3_135: now also U4.39 (PB3/I2S1_CK/SPI1_SCK/TIM2_CH2/TSC_G5_IO1)
- net DOUT_K3_21: now also U4.26 (PB13/I2C2_SCL/I2S2_CK/SPI2_SCK/TIM1_CH1N/TSC_G6_IO3/USART3_CTS)
- net DOUT_K4_T2: now also U4.30 (DAC_EXTI9/TIM15_BKIN/TIM1_CH2/TSC_G4_IO1/USART1_TX/PA9), J18.1 (Pin_1)
- net DOUT_K5_S3: now also U4.28 (PB15/I2S2_SD/RTC_REFIN/SPI2_MOSI/SYS_WKUP7/TIM15_CH1N/TIM15_CH2/TIM1_CH3N)
- net DOUT_K6_20B: now also U4.38 (I2S1_WS/SPI1_NSS/TIM2_CH1/TIM2_ETR/USART2_RX/USART4_DE/USART4_RTS/PA15)
- net DOUT_LED_RED: now also U4.17 (ADC_IN7/COMP2_OUT/I2S1_SD/SPI1_MOSI/TIM14_CH1/TIM17_CH1/TIM1_CH1N/TIM3_CH2/TSC_G2_IO4/PA7)
- net DOUT_SW_UKN: now also U4.25 (PB12/I2S2_WS/SPI2_NSS/TIM15_BKIN/TIM1_BKIN/TSC_G6_IO2/USART3_CK)
- net GND: now also R19.1, J18.3 (Pin_3); no longer C16.2, R20.1, U3.1 (A0), U3.2 (A1), U3.3 (A2)
- net ODSW_1: now also U4.40 (PB4/I2S1_MCK/SPI1_MISO/TIM17_BKIN/TIM3_CH1/TSC_G5_IO2)
- net ODSW_2: now also U4.41 (PB5/I2C1_SMBA/I2S1_SD/SPI1_MOSI/SYS_WKUP6/TIM16_BKIN/TIM3_CH2)
- net at J16.3 (Pin_3): now also Q7.1 (A1), R28.1, R30.2; no longer U6.6
- net at J16.4 (Pin_4): now also C16.1, R20.2, Q7.2 (A2); no longer U6.4
- removed net RS422RX: U1.1 (RO), U4.31 (TIM17_BKIN/TIM1_CH3/TSC_G4_IO2/USART1_RX/PA10)
- removed net RS422TX: U1.4 (DI), U4.30 (DAC_EXTI9/TIM15_BKIN/TIM1_CH2/TSC_G4_IO1/USART1_TX/PA9)
- new net: JP3.2, U3.1 (A0)
- new net: JP2.2, U3.2 (A1)
- new net: JP1.2, U3.3 (A2)
- new net: Q7.3 (G), R20.1, U6.4
- new net: R28.2, U6.6
- new net: C16.2, R29.2
- new net: R29.1, R30.1
Other:
- moved on the sheet: U3

Commit message: Update kicad board
Parts:
- C1, C10, C11, C12, C13, C14, C15, C16, C17, C2, C3, C4, C5, C6, C7, C8, C9: symbol C -> base_heating-rescue:C
- D1, D2: symbol LED -> base_heating-rescue:LED
- D3: symbol D_TVS_x2_AAC -> base_heating-rescue:D_TVS_x2_AAC
- D4, D5: symbol D_Zener -> base_heating-rescue:D_Zener
- J1, J2: symbol Conn_01x20_Male -> Connector:Conn_01x20_Male
- J10, J3, J8, J9: symbol Conn_01x04 -> base_heating-rescue:Conn_01x04
- J11, J18, J4, J7: symbol Conn_01x03 -> base_heating-rescue:Conn_01x03
- J12, J13, J14, J15, J16, J17, J5, J6: symbol Screw_Terminal_01x04 -> Connector:Screw_Terminal_01x04
- JP1, JP2, JP3: symbol Jumper_NO_Small -> base_heating-rescue:Jumper_NO_Small
- MK1, MK2: symbol Mounting_Hole -> base_heating-rescue:Mounting_Hole
- Q1: symbol NTR2101P -> base_heating-rescue:NTR2101P
- Q2, Q3, Q4, Q5: symbol IRF540N -> base_heating-rescue:IRF540N
- Q6, Q7: symbol BT136-800 -> base_heating-rescue:BT136-800
- R1, R10, R11, R12, R13, R14, R15, R16, R17, R18, R19, R2, R20, R21, R22, R23, R24, R25, R26, R27, R28, R29, R3, R30, R4, R5, R6, R7, R8, R9: symbol R -> base_heating-rescue:R
- U1: symbol MAX3078E -> base_heating-rescue:MAX3078E
- U2: symbol SN65HVD230 -> base_heating-rescue:SN65HVD230
- U3: symbol AT24CS64-SSHM -> base_heating-rescue:AT24CS64-SSHM
- U4: symbol STM32F072C8Tx -> base_heating-rescue:STM32F072C8Tx
- U5, U6: symbol MOC3061M -> base_heating-rescue:MOC3061M
